Commit message: add gazebo launch

File: adap2e_description/urdf/adap2e.xacro (robot description, xacro)
@@ -1,86 +1,79 @@
 <?xml version="1.0"?>
 <robot name="adap2e" xmlns:xacro="http://www.ros.org/wiki/xacro">
-  <xacro:macro name="adap2e" params="model">
-    <xacro:include filename="$(find romea_odo_description)/urdf/4WS_4WD_chassis.xacro" />
-    <xacro:include filename="$(find romea_odo_description)/ros2_control/4WS_4WD.ros2_control.xacro"/>
-    <xacro:property name="chassis_conf_file" value="$(find adap2e_description)/config/adap2e_${model}_chassis.yaml" />
-    <xacro:property name="kinematic_conf_file" value="$(find adap2e_description)/config/adap2e_${model}_kinematic.yaml" />
-    <xacro:property name="joints_conf_file" value="$(find adap2e_description)/config/adap2e_joints.yaml" />
-    <xacro:property name="links_conf_file" value="$(find adap2e_description)/config/adap2e_links.yaml" />
-    <xacro:property name="chassis_props" value="${load_yaml(chassis_conf_file)}"/>
-    <xacro:property name="kinematic_props" value="${load_yaml(kinematic_conf_file)}"/>
-    <xacro:property name="joints" value="${load_yaml(joints_conf_file)}"/>
-    <xacro:property name="links" value="${load_yaml(links_conf_file)}"/>
-    <!-- Link names -->
-    <xacro:property name="base_link" value="${links['base_link_name']}" />
-    <xacro:property name="base_footprint_link" value="${links['base_footprint_link_name']}" />
-    <xacro:property name="inertial_link" value="${links['inertial_link_name']}" />
-    <xacro:property name="front_left_wheel_steering_link" value="${links['front_left_wheel_steering_link_name']}" />
-    <xacro:property name="front_right_wheel_steering_link" value="${links['front_right_wheel_steering_link_name']}" />
-    <xacro:property name="rear_left_wheel_steering_link" value="${links['rear_left_wheel_steering_link_name']}" />
-    <xacro:property name="rear_right_wheel_steering_link" value="${links['rear_right_wheel_steering_link_name']}" />
-    <xacro:property name="front_left_wheel_spinning_link" value="${links['front_left_wheel_spinning_link_name']}" />
-    <xacro:property name="front_right_wheel_spinning_link" value="${links['front_right_wheel_spinning_link_name']}" />
-    <xacro:property name="rear_left_wheel_spinning_link" value="${links['rear_left_wheel_spinning_link_name']}" />
-    <xacro:property name="rear_right_wheel_spinning_link" value="${links['rear_right_wheel_spinning_link_name']}" />
-    <!-- Joint names -->
-    <xacro:property name="base_footprint_joint" value="${joints['base_footprint_joint_name']}" />
-    <xacro:property name="inertial_joint" value="${joints['inertial_joint_name']}" />
-    <xacro:property name="front_left_wheel_steering_joint" value="${joints['front_left_wheel_steering_joint_name']}" />
-    <xacro:property name="front_right_wheel_steering_joint" value="${joints['front_right_wheel_steering_joint_name']}" />
-    <xacro:property name="rear_left_wheel_steering_joint" value="${joints['rear_left_wheel_steering_joint_name']}" />
-    <xacro:property name="rear_right_wheel_steering_joint" value="${joints['rear_right_wheel_steering_joint_name']}" />
-    <xacro:property name="front_left_wheel_spinning_joint" value="${joints['front_left_wheel_spinning_joint_name']}" />
-    <xacro:property name="front_right_wheel_spinning_joint" value="${joints['front_right_wheel_spinning_joint_name']}" />
-    <xacro:property name="rear_left_wheel_spinning_joint" value="${joints['rear_left_wheel_spinning_joint_name']}" />
-    <xacro:property name="rear_right_wheel_spinning_joint" value="${joints['rear_right_wheel_spinning_joint_name']}" />
-    <!-- Base Properties -->
-    <xacro:property name="aabb_length" value="${chassis_props['aabb']['length']}" />
-    <xacro:property name="aabb_width" value="${chassis_props['aabb']['width']}" />
-    <xacro:property name="aabb_height" value="${chassis_props['aabb']['height']}" />
-    <xacro:property name="wheelbase" value="${chassis_props['wheelbase']}"/>
-    <xacro:property name="front_track" value="${chassis_props['wheel_track']['front']}"/>
-    <xacro:property name="rear_track" value="${chassis_props['wheel_track']['rear']}"/>
-    <xacro:property name="mass_base" value="15" />
-<!--    <xacro:property name="mass_base" value="${chassis_props['mass']}" />-->
-    <xacro:property name="mass_center_x" value="${chassis_props['mass_center_position'][0]}" />
-    <xacro:property name="mass_center_y" value="${chassis_props['mass_center_position'][1]}" />
-    <xacro:property name="mass_center_z" value="${chassis_props['mass_center_position'][2]}" />
-    <xacro:property name="minimal_wheel_steering_angle" value="-${kinematic_props['maximal_wheel_angle']}"/>
-    <xacro:property name="maximal_wheel_steering_angle" value="${kinematic_props['maximal_wheel_angle']}"/>
-    <xacro:property name="maximal_wheel_speed" value="${kinematic_props['maximal_wheel_speed']}"/>
-    <xacro:property name="body_reference_x" value="${kinematic_props['body_reference_x']}" />
-    <!-- Wheel Properties -->
-    <xacro:property name="steering_link_mass" value="3" />
-    <xacro:property name="steering_link_y" value="0.05" />
-    <xacro:property name="steering_link_xz" value="0.1" />
-    <xacro:property name="front_wheel_radius" value="${chassis_props['wheel_radius']['front']}" />
-    <xacro:property name="rear_wheel_radius" value="${chassis_props['wheel_radius']['rear']}" />
-    <xacro:property name="front_wheel_width" value="${chassis_props['wheel_width']['front']}" />
-    <xacro:property name="rear_wheel_width" value="${chassis_props['wheel_width']['rear']}" />
-    <xacro:property name="front_wheel_mass" value="10" />
-    <xacro:property name="rear_wheel_mass" value="10" />
-    <!-- Wheel Mounting Positions -->
-    <xacro:property name="ground_clearance" value="${chassis_props['ground_clearance']}"/>
-    <xacro:property name="front_wheel_y_offset" value="${chassis_props['hub_carrier_offset']['front']}" />
-    <xacro:property name="rear_wheel_y_offset" value="${chassis_props['hub_carrier_offset']['rear']}" />
-    <xacro:property name="chassis_height" value="${min(front_wheel_radius,rear_wheel_radius)}" />
-    <!-- visual chassis -->
-    <xacro:chassis>
-     <visual>
-       <origin xyz="${-body_reference_x} 0 ${chassis_height}" rpy="0 0 ${M_PI/2.0}" />
-       <geometry>
-         <mesh filename="package://adap2e_description/meshes/framev3_05.dae"/>
-       </geometry>
-       <material name="grey">
-         <color rgba="0.6 0.6 0.6 1"/>
-       </material>
-    </visual>
-    <!-- steering geometry -->
-    <box size="0.05 ${steering_link_y} 0.05"/>
-    <!-- wheel geometry -->
-    <mesh filename="package://adap2e_description/meshes/wheel_02.dae"/>
-    </xacro:chassis>
-    <xacro:base_control/>
+    <xacro:macro name="adap2e" params="model use_sim prefix">
+      <xacro:include filename="$(find romea_mobile_base_description)/urdf/4WS_4WD_chassis.xacro" />
+      <xacro:include filename="$(find romea_mobile_base_description)/ros2_control/4WS_4WD.ros2_control.xacro"/>
+      <xacro:property name="conf" value="$(find adap2e_description)/config/adap2e_${model}.yaml" />
+      <xacro:property name="props" value="${load_yaml(conf)['/**']['ros__parameters']['base_info']}" />
+      <!-- Link names -->
+      <xacro:property name="base_link" value="${props['links']['base_link_name']}" />
+      <xacro:property name="base_footprint_link" value="${props['links']['base_footprint_link_name']}" />
+      <xacro:property name="inertial_link" value="${props['links']['inertial_link_name']}" />
+      <xacro:property name="front_left_wheel_steering_link" value="${props['links']['front_left_wheel_steering_link_name']}" />
+      <xacro:property name="front_right_wheel_steering_link" value="${props['links']['front_right_wheel_steering_link_name']}" />
+      <xacro:property name="rear_left_wheel_steering_link" value="${props['links']['rear_left_wheel_steering_link_name']}" />
+      <xacro:property name="rear_right_wheel_steering_link" value="${props['links']['rear_right_wheel_steering_link_name']}" />
+      <xacro:property name="front_left_wheel_spinning_link" value="${props['links']['front_left_wheel_spinning_link_name']}" />
+      <xacro:property name="front_right_wheel_spinning_link" value="${props['links']['front_right_wheel_spinning_link_name']}" />
+      <xacro:property name="rear_left_wheel_spinning_link" value="${props['links']['rear_left_wheel_spinning_link_name']}" />
+      <xacro:property name="rear_right_wheel_spinning_link" value="${props['links']['rear_right_wheel_spinning_link_name']}" />
+      <!-- Joint names -->
+      <xacro:property name="base_footprint_joint" value="${props['joints']['base_footprint_joint_name']}" />
+      <xacro:property name="inertial_joint" value="${props['joints']['inertial_joint_name']}" />
+      <xacro:property name="front_left_wheel_steering_joint" value="${props['joints']['front_left_wheel_steering_joint_name']}" />
+      <xacro:property name="front_right_wheel_steering_joint" value="${props['joints']['front_right_wheel_steering_joint_name']}" />
+      <xacro:property name="rear_left_wheel_steering_joint" value="${props['joints']['rear_left_wheel_steering_joint_name']}" />
+      <xacro:property name="rear_right_wheel_steering_joint" value="${props['joints']['rear_right_wheel_steering_joint_name']}" />
+      <xacro:property name="front_left_wheel_spinning_joint" value="${props['joints']['front_left_wheel_spinning_joint_name']}" />
+      <xacro:property name="front_right_wheel_spinning_joint" value="${props['joints']['front_right_wheel_spinning_joint_name']}" />
+      <xacro:property name="rear_left_wheel_spinning_joint" value="${props['joints']['rear_left_wheel_spinning_joint_name']}" />
+      <xacro:property name="rear_right_wheel_spinning_joint" value="${props['joints']['rear_right_wheel_spinning_joint_name']}" />
+      <!-- Base Properties -->
+      <xacro:property name="aabb_length" value="${props['geometry']['aabb']['length']}" />
+      <xacro:property name="aabb_width" value="${props['geometry']['aabb']['width']}" />
+      <xacro:property name="aabb_height" value="${props['geometry']['aabb']['height']}" />
+      <xacro:property name="wheelbase" value="${props['geometry']['axles_distance']}"/>
+      <xacro:property name="front_track" value="${props['geometry']['front_axle']['wheels_distance']}"/>
+      <xacro:property name="rear_track" value="${props['geometry']['rear_axle']['wheels_distance']}"/>
+      <xacro:property name="mass_base" value="${props['inertia']['mass']}" />
+      <xacro:property name="mass_center_x" value="${props['inertia']['center'][0]}" />
+      <xacro:property name="mass_center_y" value="${props['inertia']['center'][1]}" />
+      <xacro:property name="mass_center_z" value="${props['inertia']['center'][2]}" />
+      <xacro:property name="minimal_wheel_steering_angle" value="-${props['wheels_steering_control']['command']['maximal_angle']}"/>
+      <xacro:property name="maximal_wheel_steering_angle" value="${props['wheels_steering_control']['command']['maximal_angle']}"/>
+      <xacro:property name="maximal_wheel_speed" value="${props['wheels_speed_control']['command']['maximal_speed']}"/>
+      <xacro:property name="body_reference_x" value="${props['control_point'][0]}" />
+      <!-- Wheel Properties -->
+      <xacro:property name="steering_link_mass" value="3" />
+      <xacro:property name="steering_link_y" value="0.05" />
+      <xacro:property name="steering_link_xz" value="0.1" />
+      <xacro:property name="front_wheel_radius" value="${props['geometry']['front_axle']['wheels']['radius']}" />
+      <xacro:property name="rear_wheel_radius" value="${props['geometry']['rear_axle']['wheels']['radius']}" />
+      <xacro:property name="front_wheel_width" value="${props['geometry']['front_axle']['wheels']['width']}" />
+      <xacro:property name="rear_wheel_width" value="${props['geometry']['rear_axle']['wheels']['width']}" />
+      <xacro:property name="front_wheel_mass" value="10" />
+      <xacro:property name="rear_wheel_mass" value="10" />
+      <!-- Wheel Mounting Positions -->
+      <xacro:property name="ground_clearance" value="${props['geometry']['ground_clearance']}"/>
+      <xacro:property name="front_wheel_y_offset" value="${props['geometry']['front_axle']['wheels']['hub_carrier_offset']}" />
+      <xacro:property name="rear_wheel_y_offset" value="${props['geometry']['rear_axle']['wheels']['hub_carrier_offset']}" />
+      <xacro:property name="chassis_height" value="${min(front_wheel_radius,rear_wheel_radius)}" />
+      <!-- visual chassis -->
+      <xacro:chassis>
+         <visual>
+           <origin xyz="${-body_reference_x} 0 ${chassis_height}" rpy="0 0 ${M_PI/2.0}" />
+           <geometry>
+             <mesh filename="package://adap2e_description/meshes/framev3_05.dae"/>
+           </geometry>
+           <material name="grey">
+             <color rgba="0.6 0.6 0.6 1"/>
+           </material>
+        </visual>
+        <!-- steering geometry -->
+        <box size="0.05 ${steering_link_y} 0.05"/>
+        <!-- wheel geometry -->
+        <mesh filename="package://adap2e_description/meshes/wheel_02.dae"/>
+      </xacro:chassis>
+     <xacro:base_control use_sim="${use_sim}"/>
   </xacro:macro>
 </robot>

File: adap2e_description/urdf/adap2e_fat.urdf.xacro (robot description, xacro)
@@ -1,11 +1,12 @@
 <?xml version='1.0' encoding='utf-8'?>
 <robot name="adap2e_fat" xmlns:xacro="http://www.ros.org/wiki/xacro">
-  <xacro:property name="prefix" value="" />
+  <xacro:arg name="prefix" default="" />
+  <xacro:arg name="use_sim" default="true" />
+  <xacro:arg name="controller_conf_yaml_file" default=""/>
   <xacro:include filename="$(find adap2e_description)/urdf/adap2e.xacro" />
-  <xacro:adap2e model="fat"/>
+  <xacro:adap2e model="fat" use_sim="$(arg use_sim)" prefix="$(arg prefix)"/>
   <gazebo>
-    <plugin filename="libgazebo_ros_control.so" name="gazebo_ros_control">
-    <robotSimType>gazebo_ros_control/DefaultRobotHWSim</robotSimType>
-    <legacyModeNS>false</legacyModeNS>
+    <plugin filename="libgazebo_ros2_control.so" name="gazebo_ros2_control">
+           <parameters>$(arg controller_conf_yaml_file)</parameters>
     </plugin>
   </gazebo>

File: adap2e_description/urdf/adap2e_slim.urdf.xacro (robot description, xacro)
@@ -1,11 +1,12 @@
 <?xml version='1.0' encoding='utf-8'?>
-<robot name="adap2e_slim" xmlns:xacro="http://www.ros.org/wiki/xacro">
-  <xacro:property name="prefix" value="" />
+<robot name="adap2e_fat" xmlns:xacro="http://www.ros.org/wiki/xacro">
+  <xacro:arg name="prefix" default="" />
+  <xacro:arg name="use_sim" default="true" />
+  <xacro:arg name="controller_conf_yaml_file" default=""/>
   <xacro:include filename="$(find adap2e_description)/urdf/adap2e.xacro" />
-  <xacro:adap2e model="slim"/>
+  <xacro:adap2e model="slim" use_sim="$(arg use_sim)" prefix="$(arg prefix)"/>
   <gazebo>
-    <plugin filename="libgazebo_ros_control.so" name="gazebo_ros_control">
-    <robotSimType>gazebo_ros_control/DefaultRobotHWSim</robotSimType>
-    <legacyModeNS>false</legacyModeNS>
+    <plugin filename="libgazebo_ros2_control.so" name="gazebo_ros2_control">
+           <parameters>$(arg controller_conf_yaml_file)</parameters>
     </plugin>
   </gazebo>

Commit message: adap2e description : refactoring due to changes in mobile base description package

File: adap2e_description/urdf/adap2e.xacro (robot description, xacro)
@@ -1,5 +1,5 @@
 <?xml version="1.0"?>
 <robot name="adap2e" xmlns:xacro="http://www.ros.org/wiki/xacro">
-    <xacro:macro name="adap2e" params="model use_sim prefix">
+    <xacro:macro name="adap2e" params="model mode prefix">
       <xacro:include filename="$(find romea_mobile_base_description)/urdf/4WS_4WD_chassis.xacro" />
       <xacro:include filename="$(find romea_mobile_base_description)/ros2_control/4WS_4WD.ros2_control.xacro"/>
@@ -59,4 +59,7 @@
       <xacro:property name="rear_wheel_y_offset" value="${props['geometry']['rear_axle']['wheels']['hub_carrier_offset']}" />
       <xacro:property name="chassis_height" value="${min(front_wheel_radius,rear_wheel_radius)}" />
+      <!-- Ros2 control hardware plugin -->
+      <xacro:property name="simulation_hardware_plugin" value="romea_mobile_base_gazebo/GazeboSystemInterface4WS4WD"/>
+      <xacro:property name="live_hardware_plugin" value="adap2e_hardware/Adap2eHardware"/>
       <!-- visual chassis -->
       <xacro:chassis>
@@ -75,5 +78,5 @@
         <mesh filename="package://adap2e_description/meshes/wheel_02.dae"/>
       </xacro:chassis>
-     <xacro:base_control use_sim="${use_sim}"/>
+     <xacro:base_control mode="${mode}"/>
   </xacro:macro>
 </robot>

File: adap2e_description/urdf/adap2e_fat.urdf.xacro (robot description, xacro)
@@ -2,8 +2,8 @@
 <robot name="adap2e_fat" xmlns:xacro="http://www.ros.org/wiki/xacro">
   <xacro:arg name="prefix" default="" />
-  <xacro:arg name="use_sim" default="true" />
+  <xacro:arg name="mode" default="simulation" />
   <xacro:arg name="controller_conf_yaml_file" default=""/>
   <xacro:include filename="$(find adap2e_description)/urdf/adap2e.xacro" />
-  <xacro:adap2e model="fat" use_sim="$(arg use_sim)" prefix="$(arg prefix)"/>
+  <xacro:adap2e model="fat" mode="$(arg mode)" prefix="$(arg prefix)"/>
   <gazebo>
     <plugin filename="libgazebo_ros2_control.so" name="gazebo_ros2_control">

File: adap2e_description/urdf/adap2e_slim.urdf.xacro (robot description, xacro)
@@ -2,8 +2,8 @@
 <robot name="adap2e_fat" xmlns:xacro="http://www.ros.org/wiki/xacro">
   <xacro:arg name="prefix" default="" />
-  <xacro:arg name="use_sim" default="true" />
+  <xacro:arg name="mode" default="simulation" />
   <xacro:arg name="controller_conf_yaml_file" default=""/>
   <xacro:include filename="$(find adap2e_description)/urdf/adap2e.xacro" />
-  <xacro:adap2e model="slim" use_sim="$(arg use_sim)" prefix="$(arg prefix)"/>
+  <xacro:adap2e model="slim" mode="$(arg mode)" prefix="$(arg prefix)"/>
   <gazebo>
     <plugin filename="libgazebo_ros2_control.so" name="gazebo_ros2_control">

Commit message: adap2e description : update xacro description

File: adap2e_description/urdf/adap2e.xacro (robot description, xacro)
@@ -33,4 +33,7 @@
       <xacro:property name="aabb_width" value="${props['geometry']['aabb']['width']}" />
       <xacro:property name="aabb_height" value="${props['geometry']['aabb']['height']}" />
+      <xacro:property name="aabb_center_x" value="${props['geometry']['aabb']['center'][0]}" />
+      <xacro:property name="aabb_center_y" value="${props['geometry']['aabb']['center'][1]}" />
+      <xacro:property name="aabb_center_z" value="${props['geometry']['aabb']['center'][2]}" />
       <xacro:property name="wheelbase" value="${props['geometry']['axles_distance']}"/>
       <xacro:property name="front_track" value="${props['geometry']['front_axle']['wheels_distance']}"/>

Commit message: fix xacro description

File: adap2e_description/urdf/adap2e.xacro (robot description, xacro)
@@ -5,5 +5,5 @@
       <xacro:include filename="$(find romea_mobile_base_description)/ros2_control/base4WS4WD.ros2_control.xacro"/>
       <xacro:property name="conf" value="$(find adap2e_description)/config/adap2e_${model}.yaml" />
-      <xacro:property name="props" value="${load_yaml(conf)['/**']['ros__parameters']['base_info']}" />
+      <xacro:property name="props" value="${load_yaml(conf)}" />
       <!-- Link names -->
       <xacro:property name="base_link" value="${props['links']['base_link_name']}" />
