Commit message: update description to take into account ros_namespace in gazebo_ros2_control plugin

File: adap2e_description/urdf/adap2e.xacro (robot description, xacro)
@@ -1,87 +1,115 @@
 <?xml version="1.0"?>
 <robot name="adap2e" xmlns:xacro="http://www.ros.org/wiki/xacro">
-    <xacro:macro name="adap2e" params="model mode prefix">
-      <xacro:include filename="$(find romea_mobile_base_description)/urdf/base4WS4WD.chassis.xacro" />
-      <xacro:include filename="$(find romea_mobile_base_description)/ros2_control/base4WS4WD.ros2_control.xacro"/>
-      <xacro:property name="conf" value="$(find adap2e_description)/config/adap2e_${model}.yaml" />
-      <xacro:property name="props" value="${load_yaml(conf)}" />
-      <!-- Link names -->
-      <xacro:property name="base_link" value="${props['links']['base_link_name']}" />
-      <xacro:property name="base_footprint_link" value="${props['links']['base_footprint_link_name']}" />
-      <xacro:property name="inertial_link" value="${props['links']['inertial_link_name']}" />
-      <xacro:property name="front_left_wheel_steering_link" value="${props['links']['front_left_wheel_steering_link_name']}" />
-      <xacro:property name="front_right_wheel_steering_link" value="${props['links']['front_right_wheel_steering_link_name']}" />
-      <xacro:property name="rear_left_wheel_steering_link" value="${props['links']['rear_left_wheel_steering_link_name']}" />
-      <xacro:property name="rear_right_wheel_steering_link" value="${props['links']['rear_right_wheel_steering_link_name']}" />
-      <xacro:property name="front_left_wheel_spinning_link" value="${props['links']['front_left_wheel_spinning_link_name']}" />
-      <xacro:property name="front_right_wheel_spinning_link" value="${props['links']['front_right_wheel_spinning_link_name']}" />
-      <xacro:property name="rear_left_wheel_spinning_link" value="${props['links']['rear_left_wheel_spinning_link_name']}" />
-      <xacro:property name="rear_right_wheel_spinning_link" value="${props['links']['rear_right_wheel_spinning_link_name']}" />
-      <!-- Joint names -->
-      <xacro:property name="base_footprint_joint" value="${props['joints']['base_footprint_joint_name']}" />
-      <xacro:property name="inertial_joint" value="${props['joints']['inertial_joint_name']}" />
-      <xacro:property name="front_left_wheel_steering_joint" value="${props['joints']['front_left_wheel_steering_joint_name']}" />
-      <xacro:property name="front_right_wheel_steering_joint" value="${props['joints']['front_right_wheel_steering_joint_name']}" />
-      <xacro:property name="rear_left_wheel_steering_joint" value="${props['joints']['rear_left_wheel_steering_joint_name']}" />
-      <xacro:property name="rear_right_wheel_steering_joint" value="${props['joints']['rear_right_wheel_steering_joint_name']}" />
-      <xacro:property name="front_left_wheel_spinning_joint" value="${props['joints']['front_left_wheel_spinning_joint_name']}" />
-      <xacro:property name="front_right_wheel_spinning_joint" value="${props['joints']['front_right_wheel_spinning_joint_name']}" />
-      <xacro:property name="rear_left_wheel_spinning_joint" value="${props['joints']['rear_left_wheel_spinning_joint_name']}" />
-      <xacro:property name="rear_right_wheel_spinning_joint" value="${props['joints']['rear_right_wheel_spinning_joint_name']}" />
-      <!-- Base Properties -->
-      <xacro:property name="aabb_length" value="${props['geometry']['aabb']['length']}" />
-      <xacro:property name="aabb_width" value="${props['geometry']['aabb']['width']}" />
-      <xacro:property name="aabb_height" value="${props['geometry']['aabb']['height']}" />
-      <xacro:property name="aabb_center_x" value="${props['geometry']['aabb']['center'][0]}" />
-      <xacro:property name="aabb_center_y" value="${props['geometry']['aabb']['center'][1]}" />
-      <xacro:property name="aabb_center_z" value="${props['geometry']['aabb']['center'][2]}" />
-      <xacro:property name="wheelbase" value="${props['geometry']['axles_distance']}"/>
-      <xacro:property name="front_track" value="${props['geometry']['front_axle']['wheels_distance']}"/>
-      <xacro:property name="rear_track" value="${props['geometry']['rear_axle']['wheels_distance']}"/>
-      <xacro:property name="mass_base" value="${props['inertia']['mass']}" />
-      <xacro:property name="mass_center_x" value="${props['inertia']['center'][0]}" />
-      <xacro:property name="mass_center_y" value="${props['inertia']['center'][1]}" />
-      <xacro:property name="mass_center_z" value="${props['inertia']['center'][2]}" />
-      <xacro:property name="minimal_wheel_steering_angle" value="-${props['wheels_steering_control']['command']['maximal_angle']}"/>
-      <xacro:property name="maximal_wheel_steering_angle" value="${props['wheels_steering_control']['command']['maximal_angle']}"/>
-      <xacro:property name="maximal_wheel_speed" value="${props['wheels_speed_control']['command']['maximal_speed']}"/>
-      <xacro:property name="body_reference_x" value="${props['control_point'][0]}" />
-      <!-- Wheel Properties -->
-      <xacro:property name="steering_link_mass" value="3" />
-      <xacro:property name="steering_link_y" value="0.05" />
-      <xacro:property name="steering_link_xz" value="0.1" />
-      <xacro:property name="front_wheel_radius" value="${props['geometry']['front_axle']['wheels']['radius']}" />
-      <xacro:property name="rear_wheel_radius" value="${props['geometry']['rear_axle']['wheels']['radius']}" />
-      <xacro:property name="front_wheel_width" value="${props['geometry']['front_axle']['wheels']['width']}" />
-      <xacro:property name="rear_wheel_width" value="${props['geometry']['rear_axle']['wheels']['width']}" />
-      <xacro:property name="front_wheel_mass" value="10" />
-      <xacro:property name="rear_wheel_mass" value="10" />
-      <!-- Wheel Mounting Positions -->
-      <xacro:property name="ground_clearance" value="${props['geometry']['ground_clearance']}"/>
-      <xacro:property name="front_wheel_y_offset" value="${props['geometry']['front_axle']['wheels']['hub_carrier_offset']}" />
-      <xacro:property name="rear_wheel_y_offset" value="${props['geometry']['rear_axle']['wheels']['hub_carrier_offset']}" />
-      <xacro:property name="chassis_height" value="${min(front_wheel_radius,rear_wheel_radius)}" />
-      <!-- Ros2 control hardware plugin -->
-      <xacro:property name="simulation_hardware_plugin" value="romea_mobile_base_gazebo/GazeboSystemInterface4WS4WD"/>
-      <xacro:property name="live_hardware_plugin" value="adap2e_hardware/Adap2eHardware"/>
-      <!-- visual chassis -->
-      <xacro:chassis>
-         <visual>
-           <origin xyz="${-body_reference_x} 0 ${chassis_height}" rpy="0 0 ${M_PI/2.0}" />
-           <geometry>
-             <mesh filename="package://adap2e_description/meshes/framev3_05.dae"/>
-           </geometry>
-           <material name="grey">
-             <color rgba="0.6 0.6 0.6 1"/>
-           </material>
-        </visual>
-        <!-- steering geometry -->
-        <box size="0.05 ${steering_link_y} 0.05"/>
-        <!-- wheel geometry -->
-        <mesh filename="package://adap2e_description/meshes/wheel_02.dae"/>
-      </xacro:chassis>
-     <xacro:if value="${mode == 'simulation' or mode == 'live'}">
-        <xacro:base_control mode="${mode}"/>
-     </xacro:if>
+  <xacro:macro name="adap2e" params="model mode prefix">
+    <xacro:include filename="$(find romea_mobile_base_description)/urdf/base4WS4WD.chassis.xacro" />
+    <xacro:include
+      filename="$(find romea_mobile_base_description)/ros2_control/base4WS4WD.ros2_control.xacro" />
+    <xacro:property name="conf" value="$(find adap2e_description)/config/adap2e_${model}.yaml" />
+    <xacro:property name="props" value="${load_yaml(conf)}" />
+    <!-- Link names -->
+    <xacro:property name="base_link" value="${props['links']['base_link_name']}" />
+    <xacro:property name="base_footprint_link" value="${props['links']['base_footprint_link_name']}" />
+    <xacro:property name="inertial_link" value="${props['links']['inertial_link_name']}" />
+    <xacro:property name="front_left_wheel_steering_link"
+      value="${props['links']['front_left_wheel_steering_link_name']}" />
+    <xacro:property name="front_right_wheel_steering_link"
+      value="${props['links']['front_right_wheel_steering_link_name']}" />
+    <xacro:property name="rear_left_wheel_steering_link"
+      value="${props['links']['rear_left_wheel_steering_link_name']}" />
+    <xacro:property name="rear_right_wheel_steering_link"
+      value="${props['links']['rear_right_wheel_steering_link_name']}" />
+    <xacro:property name="front_left_wheel_spinning_link"
+      value="${props['links']['front_left_wheel_spinning_link_name']}" />
+    <xacro:property name="front_right_wheel_spinning_link"
+      value="${props['links']['front_right_wheel_spinning_link_name']}" />
+    <xacro:property name="rear_left_wheel_spinning_link"
+      value="${props['links']['rear_left_wheel_spinning_link_name']}" />
+    <xacro:property name="rear_right_wheel_spinning_link"
+      value="${props['links']['rear_right_wheel_spinning_link_name']}" />
+    <!-- Joint names -->
+    <xacro:property name="base_footprint_joint"
+      value="${props['joints']['base_footprint_joint_name']}" />
+    <xacro:property name="inertial_joint" value="${props['joints']['inertial_joint_name']}" />
+    <xacro:property name="front_left_wheel_steering_joint"
+      value="${props['joints']['front_left_wheel_steering_joint_name']}" />
+    <xacro:property name="front_right_wheel_steering_joint"
+      value="${props['joints']['front_right_wheel_steering_joint_name']}" />
+    <xacro:property name="rear_left_wheel_steering_joint"
+      value="${props['joints']['rear_left_wheel_steering_joint_name']}" />
+    <xacro:property name="rear_right_wheel_steering_joint"
+      value="${props['joints']['rear_right_wheel_steering_joint_name']}" />
+    <xacro:property name="front_left_wheel_spinning_joint"
+      value="${props['joints']['front_left_wheel_spinning_joint_name']}" />
+    <xacro:property name="front_right_wheel_spinning_joint"
+      value="${props['joints']['front_right_wheel_spinning_joint_name']}" />
+    <xacro:property name="rear_left_wheel_spinning_joint"
+      value="${props['joints']['rear_left_wheel_spinning_joint_name']}" />
+    <xacro:property name="rear_right_wheel_spinning_joint"
+      value="${props['joints']['rear_right_wheel_spinning_joint_name']}" />
+    <!-- Base Properties -->
+    <xacro:property name="aabb_length" value="${props['geometry']['aabb']['length']}" />
+    <xacro:property name="aabb_width" value="${props['geometry']['aabb']['width']}" />
+    <xacro:property name="aabb_height" value="${props['geometry']['aabb']['height']}" />
+    <xacro:property name="aabb_center_x" value="${props['geometry']['aabb']['center'][0]}" />
+    <xacro:property name="aabb_center_y" value="${props['geometry']['aabb']['center'][1]}" />
+    <xacro:property name="aabb_center_z" value="${props['geometry']['aabb']['center'][2]}" />
+    <xacro:property name="wheelbase" value="${props['geometry']['axles_distance']}" />
+    <xacro:property name="front_track" value="${props['geometry']['front_axle']['wheels_distance']}" />
+    <xacro:property name="rear_track" value="${props['geometry']['rear_axle']['wheels_distance']}" />
+    <xacro:property name="mass_base" value="${props['inertia']['mass']}" />
+    <xacro:property name="mass_center_x" value="${props['inertia']['center'][0]}" />
+    <xacro:property name="mass_center_y" value="${props['inertia']['center'][1]}" />
+    <xacro:property name="mass_center_z" value="${props['inertia']['center'][2]}" />
+    <xacro:property name="minimal_wheel_steering_angle"
+      value="-${props['wheels_steering_control']['command']['maximal_angle']}" />
+    <xacro:property name="maximal_wheel_steering_angle"
+      value="${props['wheels_steering_control']['command']['maximal_angle']}" />
+    <xacro:property name="maximal_wheel_speed"
+      value="${props['wheels_speed_control']['command']['maximal_speed']}" />
+    <xacro:property name="body_reference_x" value="${props['control_point'][0]}" />
+    <!-- Wheel Properties -->
+    <xacro:property name="steering_link_mass" value="3" />
+    <xacro:property name="steering_link_y" value="0.05" />
+    <xacro:property name="steering_link_xz" value="0.1" />
+    <xacro:property name="front_wheel_radius"
+      value="${props['geometry']['front_axle']['wheels']['radius']}" />
+    <xacro:property name="rear_wheel_radius"
+      value="${props['geometry']['rear_axle']['wheels']['radius']}" />
+    <xacro:property name="front_wheel_width"
+      value="${props['geometry']['front_axle']['wheels']['width']}" />
+    <xacro:property name="rear_wheel_width"
+      value="${props['geometry']['rear_axle']['wheels']['width']}" />
+    <xacro:property name="front_wheel_mass" value="10" />
+    <xacro:property name="rear_wheel_mass" value="10" />
+    <!-- Wheel Mounting Positions -->
+    <xacro:property name="ground_clearance" value="${props['geometry']['ground_clearance']}" />
+    <xacro:property name="front_wheel_y_offset"
+      value="${props['geometry']['front_axle']['wheels']['hub_carrier_offset']}" />
+    <xacro:property name="rear_wheel_y_offset"
+      value="${props['geometry']['rear_axle']['wheels']['hub_carrier_offset']}" />
+    <xacro:property name="chassis_height" value="${min(front_wheel_radius,rear_wheel_radius)}" />
+    <!-- Ros2 control hardware plugin -->
+    <xacro:property name="simulation_hardware_plugin"
+      value="romea_mobile_base_gazebo/GazeboSystemInterface4WS4WD" />
+    <xacro:property name="live_hardware_plugin" value="adap2e_hardware/Adap2eHardware" />
+    <!-- visual chassis -->
+    <xacro:chassis>
+      <visual>
+        <origin xyz="${-body_reference_x} 0 ${chassis_height}" rpy="0 0 ${M_PI/2.0}" />
+        <geometry>
+          <mesh filename="package://adap2e_description/meshes/framev3_05.dae" />
+        </geometry>
+        <material name="grey">
+          <color rgba="0.6 0.6 0.6 1" />
+        </material>
+      </visual>
+      <!-- steering geometry -->
+      <box size="0.05 ${steering_link_y} 0.05" />
+      <!-- wheel geometry -->
+      <mesh filename="package://adap2e_description/meshes/wheel_02.dae" />
+    </xacro:chassis>
+    <xacro:if value="${mode == 'simulation' or mode == 'live'}">
+      <xacro:base_control mode="${mode}" />
+    </xacro:if>
   </xacro:macro>
 </robot>

File: adap2e_description/urdf/adap2e_fat.urdf.xacro (robot description, xacro)
@@ -3,10 +3,14 @@
   <xacro:arg name="prefix" default="adap2e_" />
   <xacro:arg name="mode" default="simulation" />
-  <xacro:arg name="controller_conf_yaml_file" default=""/>
+  <xacro:arg name="controller_conf_yaml_file" default="" />
+  <xacro:arg name="ros_namespace" default="/adap2e" />
   <xacro:include filename="$(find adap2e_description)/urdf/adap2e.xacro" />
-  <xacro:adap2e model="fat" mode="$(arg mode)" prefix="$(arg prefix)"/>
+  <xacro:adap2e model="fat" mode="$(arg mode)" prefix="$(arg prefix)" />
   <gazebo>
     <plugin filename="libgazebo_ros2_control.so" name="gazebo_ros2_control">
-           <parameters>$(arg controller_conf_yaml_file)</parameters>
+      <parameters>$(arg controller_conf_yaml_file)</parameters>
+      <ros>
+        <namespace>$(arg ros_namespace)</namespace>
+      </ros>
     </plugin>
   </gazebo>

File: adap2e_description/urdf/adap2e_slim.urdf.xacro (robot description, xacro)
@@ -3,10 +3,14 @@
   <xacro:arg name="prefix" default="adap2e" />
   <xacro:arg name="mode" default="simulation" />
-  <xacro:arg name="controller_conf_yaml_file" default=""/>
+  <xacro:arg name="controller_conf_yaml_file" default="" />
+  <xacro:arg name="ros_namespace" default="/adap2e" />
   <xacro:include filename="$(find adap2e_description)/urdf/adap2e.xacro" />
-  <xacro:adap2e model="slim" mode="$(arg mode)" prefix="$(arg prefix)"/>
+  <xacro:adap2e model="slim" mode="$(arg mode)" prefix="$(arg prefix)" />
   <gazebo>
     <plugin filename="libgazebo_ros2_control.so" name="gazebo_ros2_control">
-       <parameters>$(arg controller_conf_yaml_file)</parameters>
+      <parameters>$(arg controller_conf_yaml_file)</parameters>
+      <ros>
+        <namespace>$(arg ros_namespace)</namespace>
+      </ros>
     </plugin>
   </gazebo>

Commit message: split gazebo urdf gazebo / urdf ros2 control add romea_gazebo_ros2_control gazebo plugin add possiblity to change base_name
Signed-off-by: jean.laneurit <jean.laneurit@inrae.fr>

File: adap2e_description/urdf/adap2e.xacro (robot description, xacro)
@@ -3,6 +3,6 @@
   <xacro:macro name="adap2e" params="model mode prefix">
     <xacro:include filename="$(find romea_mobile_base_description)/urdf/base4WS4WD.chassis.xacro" />
-    <xacro:include
-      filename="$(find romea_mobile_base_description)/ros2_control/base4WS4WD.ros2_control.xacro" />
+    <!-- <xacro:include
+      filename="$(find romea_mobile_base_description)/ros2_control/base4WS4WD.ros2_control.xacro" /> -->
     <xacro:property name="conf" value="$(find adap2e_description)/config/adap2e_${model}.yaml" />
     <xacro:property name="props" value="${load_yaml(conf)}" />
@@ -90,7 +90,8 @@
     <xacro:property name="chassis_height" value="${min(front_wheel_radius,rear_wheel_radius)}" />
     <!-- Ros2 control hardware plugin -->
-    <xacro:property name="simulation_hardware_plugin"
+    <!-- <xacro:property name="simulation_hardware_plugin"
       value="romea_mobile_base_gazebo/GazeboSystemInterface4WS4WD" />
-    <xacro:property name="live_hardware_plugin" value="adap2e_hardware/Adap2eHardware" />
+    <xacro:property name="live_hardware_plugin"
+      value="adap2e_hardware/Adap2eHardware" /> -->
     <!-- visual chassis -->
     <xacro:chassis>
@@ -109,7 +110,7 @@
       <mesh filename="package://adap2e_description/meshes/wheel_02.dae" />
     </xacro:chassis>
-    <xacro:if value="${mode == 'simulation' or mode == 'live'}">
+    <!-- <xacro:if value="${mode == 'simulation' or mode == 'live'}">
       <xacro:base_control mode="${mode}" />
-    </xacro:if>
+    </xacro:if> -->
   </xacro:macro>
 </robot>

File: adap2e_description/urdf/adap2e_fat.urdf.xacro (robot description, xacro)
@@ -3,15 +3,16 @@
   <xacro:arg name="prefix" default="adap2e_" />
   <xacro:arg name="mode" default="simulation" />
-  <xacro:arg name="controller_conf_yaml_file" default="" />
+  <xacro:arg name="base_name" default="base" />
+  <xacro:arg name="controller_manager_config_yaml_file" default="" />
+  <xacro:arg name="ros2_control_config_urdf_file" default="" />
   <xacro:arg name="ros_prefix" default="/adap2e/" />
   <xacro:include filename="$(find adap2e_description)/urdf/adap2e.xacro" />
   <xacro:adap2e model="fat" mode="$(arg mode)" prefix="$(arg prefix)" />
   <gazebo>
-    <plugin filename="libgazebo_ros2_control.so" name="gazebo_ros2_control">
-      <hardware>$(arg prefix)base</hardware>
-      <robot_param_node>$(arg ros_prefix)robot_state_publisher</robot_param_node>
-      <parameters>$(arg controller_conf_yaml_file)</parameters>
+    <plugin filename="libromea_gazebo_ros2_control.so" name="gazebo_ros2_control">
+      <ros2_control_config_file>$(arg ros2_control_config_urdf_file)</ros2_control_config_file>
+      <controller_manager_config_file>$(arg controller_manager_config_yaml_file)</controller_manager_config_file>
       <ros>
-        <namespace>$(arg ros_prefix)base</namespace>
+        <namespace>$(arg ros_prefix)$(arg base_name)</namespace>
       </ros>
     </plugin>

File: adap2e_description/urdf/adap2e_slim.urdf.xacro (robot description, xacro)
@@ -3,15 +3,16 @@
   <xacro:arg name="prefix" default="adap2e" />
   <xacro:arg name="mode" default="simulation" />
-  <xacro:arg name="controller_conf_yaml_file" default="" />
+  <xacro:arg name="base_name" default="base" />
+  <xacro:arg name="controller_manager_config_yaml_file" default="" />
+  <xacro:arg name="ros2_control_config_urdf_file" default="" />
   <xacro:arg name="ros_prefix" default="/adap2e/" />
   <xacro:include filename="$(find adap2e_description)/urdf/adap2e.xacro" />
   <xacro:adap2e model="slim" mode="$(arg mode)" prefix="$(arg prefix)" />
   <gazebo>
-    <plugin filename="libgazebo_ros2_control.so" name="gazebo_ros2_control">
-      <hardware>$(arg prefix)base</hardware>
-      <robot_param_node>$(arg ros_prefix)robot_state_publisher</robot_param_node>
-      <parameters>$(arg controller_conf_yaml_file)</parameters>
+    <plugin filename="libromea_gazebo_ros2_control.so" name="gazebo_ros2_control">
+      <ros2_control_config_file>$(arg ros2_control_config_urdf_file)</ros2_control_config_file>
+      <controller_manager_config_file>$(arg controller_manager_config_yaml_file)</controller_manager_config_file>
       <ros>
-        <namespace>$(arg ros_prefix)base</namespace>
+        <namespace>$(arg ros_prefix)$(arg base_name)</namespace>
       </ros>
     </plugin>

Commit message: description: remove unused lines in xacro files

File: adap2e_description/urdf/adap2e.xacro (robot description, xacro)
@@ -3,6 +3,4 @@
   <xacro:macro name="adap2e" params="model mode prefix">
     <xacro:include filename="$(find romea_mobile_base_description)/urdf/base4WS4WD.chassis.xacro" />
-    <!-- <xacro:include
-      filename="$(find romea_mobile_base_description)/ros2_control/base4WS4WD.ros2_control.xacro" /> -->
     <xacro:property name="conf" value="$(find adap2e_description)/config/adap2e_${model}.yaml" />
     <xacro:property name="props" value="${load_yaml(conf)}" />
@@ -89,9 +87,4 @@
       value="${props['geometry']['rear_axle']['wheels']['hub_carrier_offset']}" />
     <xacro:property name="chassis_height" value="${min(front_wheel_radius,rear_wheel_radius)}" />
-    <!-- Ros2 control hardware plugin -->
-    <!-- <xacro:property name="simulation_hardware_plugin"
-      value="romea_mobile_base_gazebo/GazeboSystemInterface4WS4WD" />
-    <xacro:property name="live_hardware_plugin"
-      value="adap2e_hardware/Adap2eHardware" /> -->
     <!-- visual chassis -->
     <xacro:chassis>
@@ -110,7 +103,4 @@
       <mesh filename="package://adap2e_description/meshes/wheel_02.dae" />
     </xacro:chassis>
-    <!-- <xacro:if value="${mode == 'simulation' or mode == 'live'}">
-      <xacro:base_control mode="${mode}" />
-    </xacro:if> -->
   </xacro:macro>
 </robot>
