Commit message: description: update xacro description
Signed-off-by: Jean Laneurit <jean.laneurit@inrae.fr>

File: adap2e_description/urdf/adap2e.xacro (robot description, xacro)
@@ -59,15 +59,13 @@
     <xacro:property name="mass_center_y" value="${props['inertia']['center'][1]}" />
     <xacro:property name="mass_center_z" value="${props['inertia']['center'][2]}" />
-    <xacro:property name="minimal_wheel_steering_angle"
-      value="-${props['wheels_steering_control']['command']['maximal_angle']}" />
-    <xacro:property name="maximal_wheel_steering_angle"
-      value="${props['wheels_steering_control']['command']['maximal_angle']}" />
-    <xacro:property name="maximal_wheel_speed"
-      value="${props['wheels_speed_control']['command']['maximal_speed']}" />
-    <xacro:property name="body_reference_x" value="${props['control_point'][0]}" />
-    <!-- Wheel Properties -->
-    <xacro:property name="steering_link_mass" value="3" />
-    <xacro:property name="steering_link_y" value="0.05" />
-    <xacro:property name="steering_link_xz" value="0.1" />
+    <xacro:property name="ground_clearance"
+      value="${props['geometry']['ground_clearance']}" />
+    <xacro:property name="body_reference_x"
+      value="${props['control_point'][0]}" />
+     <!-- Wheel Properties -->
+    <xacro:property name="front_hub_carrier_offset"
+      value="${props['geometry']['front_axle']['wheels']['hub_carrier_offset']}" />
+    <xacro:property name="rear_hub_carrier_offset"
+      value="${props['geometry']['rear_axle']['wheels']['hub_carrier_offset']}" />
     <xacro:property name="front_wheel_radius"
       value="${props['geometry']['front_axle']['wheels']['radius']}" />
@@ -78,15 +76,23 @@
     <xacro:property name="rear_wheel_width"
       value="${props['geometry']['rear_axle']['wheels']['width']}" />
+    <xacro:property name="maximal_wheel_speed"
+      value="${props['wheels_speed_control']['command']['maximal_speed']}" />
+    <xacro:property name="chassis_height"
+      value="${min(front_wheel_radius,rear_wheel_radius)}" />
     <xacro:property name="front_wheel_mass" value="10" />
     <xacro:property name="rear_wheel_mass" value="10" />
-    <!-- Wheel Mounting Positions -->
-    <xacro:property name="ground_clearance" value="${props['geometry']['ground_clearance']}" />
-    <xacro:property name="front_wheel_y_offset"
-      value="${props['geometry']['front_axle']['wheels']['hub_carrier_offset']}" />
-    <xacro:property name="rear_wheel_y_offset"
-      value="${props['geometry']['rear_axle']['wheels']['hub_carrier_offset']}" />
-    <xacro:property name="chassis_height" value="${min(front_wheel_radius,rear_wheel_radius)}" />
-    <!-- visual chassis -->
+    <!-- Steering Properties -->
+    <xacro:property name="minimal_wheel_steering_angle"
+      value="-${props['wheels_steering_control']['command']['maximal_angle']}" />
+    <xacro:property name="maximal_wheel_steering_angle"
+      value="${props['wheels_steering_control']['command']['maximal_angle']}" />
+    <xacro:property name="front_wheel_steering_link_mass" value="3" />
+    <xacro:property name="front_wheel_steering_link_y" value="${front_hub_carrier_offset}"/>
+    <xacro:property name="front_wheel_steering_link_xz" value="0.05" />
+    <xacro:property name="rear_wheel_steering_link_mass" value="3" />
+    <xacro:property name="rear_wheel_steering_link_y" value="${rear_hub_carrier_offset}"/>
+    <xacro:property name="rear_wheel_steering_link_xz" value="0.05" />
     <xacro:chassis>
+      <!-- visual chassis -->
       <visual>
         <origin xyz="${-body_reference_x} 0 ${chassis_height}" rpy="0 0 ${M_PI/2.0}" />
@@ -98,7 +104,11 @@
         </material>
       </visual>
-      <!-- steering geometry -->
-      <box size="0.05 ${steering_link_y} 0.05" />
-      <!-- wheel geometry -->
+      <!-- front steering link geometry -->
+      <box size="${front_wheel_steering_link_xz} ${front_wheel_steering_link_y} ${front_wheel_steering_link_xz}" />
+      <!-- front steering link geometry -->
+      <box size="${rear_wheel_steering_link_xz} ${rear_wheel_steering_link_y} ${rear_wheel_steering_link_xz}" />
+      <!-- front wheel geometry -->
+      <mesh filename="package://adap2e_description/meshes/wheel_02.dae" />
+      <!-- rear wheel geometry -->
       <mesh filename="package://adap2e_description/meshes/wheel_02.dae" />
     </xacro:chassis>

Commit message: description: update xacro file
Signed-off-by: jean.laneurit <jean.laneurit@inrae.fr>

File: adap2e_description/urdf/adap2e.xacro (robot description, xacro)
@@ -63,5 +63,5 @@
     <xacro:property name="body_reference_x"
       value="${props['control_point'][0]}" />
-     <!-- Wheel Properties -->
+    <!-- Wheel Properties -->
     <xacro:property name="front_hub_carrier_offset"
       value="${props['geometry']['front_axle']['wheels']['hub_carrier_offset']}" />
@@ -88,8 +88,8 @@
       value="${props['wheels_steering_control']['command']['maximal_angle']}" />
     <xacro:property name="front_wheel_steering_link_mass" value="3" />
-    <xacro:property name="front_wheel_steering_link_y" value="${front_hub_carrier_offset}"/>
+    <xacro:property name="front_wheel_steering_link_y" value="${front_hub_carrier_offset}" />
     <xacro:property name="front_wheel_steering_link_xz" value="0.05" />
     <xacro:property name="rear_wheel_steering_link_mass" value="3" />
-    <xacro:property name="rear_wheel_steering_link_y" value="${rear_hub_carrier_offset}"/>
+    <xacro:property name="rear_wheel_steering_link_y" value="${rear_hub_carrier_offset}" />
     <xacro:property name="rear_wheel_steering_link_xz" value="0.05" />
     <xacro:chassis>
@@ -105,7 +105,9 @@
       </visual>
       <!-- front steering link geometry -->
-      <box size="${front_wheel_steering_link_xz} ${front_wheel_steering_link_y} ${front_wheel_steering_link_xz}" />
+      <box
+        size="${front_wheel_steering_link_xz} ${front_wheel_steering_link_y} ${front_wheel_steering_link_xz}" />
       <!-- front steering link geometry -->
-      <box size="${rear_wheel_steering_link_xz} ${rear_wheel_steering_link_y} ${rear_wheel_steering_link_xz}" />
+      <box
+        size="${rear_wheel_steering_link_xz} ${rear_wheel_steering_link_y} ${rear_wheel_steering_link_xz}" />
       <!-- front wheel geometry -->
       <mesh filename="package://adap2e_description/meshes/wheel_02.dae" />

Commit message: description: change way to define visual inside xacro file
Signed-off-by: jean.laneurit <jean.laneurit@inrae.fr>

File: adap2e_description/urdf/adap2e.xacro (robot description, xacro)
@@ -3,4 +3,7 @@
   <xacro:macro name="adap2e" params="model mode prefix">
     <xacro:include filename="$(find romea_mobile_base_description)/urdf/base4WS4WD.chassis.xacro" />
+    <xacro:include filename="$(find adap2e_description)/urdf/visual/chassis.xacro" />
+    <xacro:include filename="$(find adap2e_description)/urdf/visual/wheels.xacro" />
+    <xacro:include filename="$(find adap2e_description)/urdf/visual/arms.xacro" />
     <xacro:property name="conf" value="$(find adap2e_description)/config/adap2e_${model}.yaml" />
     <xacro:property name="props" value="${load_yaml(conf)}" />
@@ -64,4 +67,6 @@
       value="${props['control_point'][0]}" />
     <!-- Wheel Properties -->
+    <xacro:property name="front_wheel_x_offset" value="0.0" />
+    <xacro:property name="rear_wheel_x_offset" value="0.0" />
     <xacro:property name="front_hub_carrier_offset"
       value="${props['geometry']['front_axle']['wheels']['hub_carrier_offset']}" />
@@ -94,24 +99,13 @@
     <xacro:property name="rear_wheel_steering_link_xz" value="0.05" />
     <xacro:chassis>
-      <!-- visual chassis -->
-      <visual>
-        <origin xyz="${-body_reference_x} 0 ${chassis_height}" rpy="0 0 ${M_PI/2.0}" />
-        <geometry>
-          <mesh filename="package://adap2e_description/meshes/framev3_05.dae" />
-        </geometry>
-        <material name="grey">
-          <color rgba="0.6 0.6 0.6 1" />
-        </material>
-      </visual>
-      <!-- front steering link geometry -->
-      <box
-        size="${front_wheel_steering_link_xz} ${front_wheel_steering_link_y} ${front_wheel_steering_link_xz}" />
-      <!-- front steering link geometry -->
-      <box
-        size="${rear_wheel_steering_link_xz} ${rear_wheel_steering_link_y} ${rear_wheel_steering_link_xz}" />
-      <!-- front wheel geometry -->
-      <mesh filename="package://adap2e_description/meshes/wheel_02.dae" />
-      <!-- rear wheel geometry -->
-      <mesh filename="package://adap2e_description/meshes/wheel_02.dae" />
+      <xacro:chassis_visual />
+      <xacro:front_left_arm_visual />
+      <xacro:front_right_arm_visual />
+      <xacro:rear_left_arm_visual />
+      <xacro:rear_right_arm_visual />
+      <xacro:front_left_wheel_visual />
+      <xacro:front_right_wheel_visual />
+      <xacro:rear_left_wheel_visual />
+      <xacro:rear_right_wheel_visual />
     </xacro:chassis>
   </xacro:macro>

Commit message: fix steering joint mass for simulation

File: adap2e_description/urdf/adap2e.xacro (robot description, xacro)
@@ -92,8 +92,8 @@
     <xacro:property name="maximal_wheel_steering_angle"
       value="${props['wheels_steering_control']['command']['maximal_angle']}" />
-    <xacro:property name="front_wheel_steering_link_mass" value="3" />
+    <xacro:property name="front_wheel_steering_link_mass" value="20" />
     <xacro:property name="front_wheel_steering_link_y" value="${front_hub_carrier_offset}" />
     <xacro:property name="front_wheel_steering_link_xz" value="0.05" />
-    <xacro:property name="rear_wheel_steering_link_mass" value="3" />
+    <xacro:property name="rear_wheel_steering_link_mass" value="20" />
     <xacro:property name="rear_wheel_steering_link_y" value="${rear_hub_carrier_offset}" />
     <xacro:property name="rear_wheel_steering_link_xz" value="0.05" />
