Commit message: add generate_ros2_control_description + use official gazebo_ros2_control plugin
Signed-off-by: jean.laneurit <jean.laneurit@inrae.fr>

File: adap2e_description/urdf/adap2e.simulation.xacro (robot description, xacro)
@@ -2,11 +2,13 @@
 <robot name="adap2e_fat" xmlns:xacro="http://www.ros.org/wiki/xacro">
   <xacro:macro name="adap2e_simulation"
-    params="mode ros_prefix base_name ros2_control_config_urdf_file controller_manager_config_yaml_file">
+    params="mode ros_prefix base_name controller_manager_config_yaml_file">
     <xacro:if value="${'simulation' in mode}">
       <xacro:if value="${'gazebo' in  mode}">
         <gazebo>
-          <plugin filename="libromea_gazebo_ros2_control.so" name="gazebo_ros2_control">
-            <ros2_control_config_file>${ros2_control_config_urdf_file}</ros2_control_config_file>
-            <controller_manager_config_file>${controller_manager_config_yaml_file}</controller_manager_config_file>
+          <plugin filename="libgazebo_ros2_control.so" name="gazebo_ros2_control">
+            <robot_param>robot_description</robot_param>
+            <robot_param_node>ros2_control_description</robot_param_node>
+            <parameters>${controller_manager_config_yaml_file}</parameters>
+            <hold_joints>true</hold_joints>
             <ros>
               <namespace>${ros_prefix}${base_name}</namespace>

File: adap2e_description/urdf/adap2e.xacro (robot description, xacro)
@@ -7,5 +7,5 @@
     <xacro:include filename="$(find adap2e_description)/urdf/visual/arms.xacro" />
     <xacro:property name="conf" value="$(find adap2e_description)/config/adap2e_${model}.yaml" />
-    <xacro:property name="props" value="${load_yaml(conf)}" />
+    <xacro:property name="props" value="${xacro.load_yaml(conf)}" />
     <!-- Link names -->
     <xacro:property name="base_link" value="${props['links']['base_link_name']}" />

File: adap2e_description/urdf/adap2e_one.urdf.xacro (robot description, xacro)
@@ -5,5 +5,4 @@
   <xacro:arg name="base_name" default="base" />
   <xacro:arg name="controller_manager_config_yaml_file" default="" />
-  <xacro:arg name="ros2_control_config_urdf_file" default="" />
   <xacro:arg name="ros_prefix" default="/adap2e/" />
   <xacro:include filename="$(find adap2e_description)/urdf/adap2e.xacro" />
@@ -17,5 +16,4 @@
     base_name="$(arg base_name)"
     ros_prefix="$(arg ros_prefix)"
-    ros2_control_config_urdf_file="$(arg ros2_control_config_urdf_file)"
     controller_manager_config_yaml_file="$(arg controller_manager_config_yaml_file)" />
 </robot>

File: adap2e_description/urdf/adap2e_two.urdf.xacro (robot description, xacro)
@@ -5,5 +5,4 @@
   <xacro:arg name="base_name" default="base" />
   <xacro:arg name="controller_manager_config_yaml_file" default="" />
-  <xacro:arg name="ros2_control_config_urdf_file" default="" />
   <xacro:arg name="ros_prefix" default="/adap2e/" />
   <xacro:include filename="$(find adap2e_description)/urdf/adap2e.xacro" />
@@ -17,5 +16,4 @@
     base_name="$(arg base_name)"
     ros_prefix="$(arg ros_prefix)"
-    ros2_control_config_urdf_file="$(arg ros2_control_config_urdf_file)"
     controller_manager_config_yaml_file="$(arg controller_manager_config_yaml_file)" />
 </robot>
