Commit message: description:  add missing properties into ros2_control xacro file
Signed-off-by: jean.laneurit <jean.laneurit@inrae.fr>

File: adap2e_description/ros2_control/adap2e.ros2_control.xacro (robot description, xacro)
@@ -34,8 +34,8 @@
     <xacro:property name="rear_wheel_radius"
       value="${props['geometry']['rear_axle']['wheels']['radius']}" />
-    <xacro:property name="front_wheel_width"
-      value="${props['geometry']['front_axle']['wheels']['width']}" />
-    <xacro:property name="rear_wheel_width"
-      value="${props['geometry']['rear_axle']['wheels']['width']}" />
+    <xacro:property name="maximal_wheel_steering_angle"
+      value="${props['wheels_steering_control']['command']['maximal_angle']}" />
+    <xacro:property name="maximal_wheel_speed"
+      value="${props['wheels_speed_control']['command']['maximal_speed']}" />
     <!-- simulation plugins -->
     <xacro:property

Commit message: add support of 4dv and isaac simulator
Signed-off-by: jean.laneurit <jean.laneurit@inrae.fr>

File: adap2e_description/ros2_control/adap2e.ros2_control.xacro (robot description, xacro)
@@ -39,10 +39,21 @@
       value="${props['wheels_speed_control']['command']['maximal_speed']}" />
     <!-- simulation plugins -->
-    <xacro:property
-      name="simulation_hardware_plugin"
-      value="romea_mobile_base_gazebo/GazeboSystemInterface4WS4WD" />
-    <xacro:property
-      name="live_hardware_plugin"
-      value="adap2e_hardware/Adap2eHardware" />
+    <xacro:if value="${'simulation' in mode}">
+      <xacro:if value="${'gazebo' in  mode}">
+        <xacro:property
+          name="simulation_hardware_plugin"
+          value="romea_mobile_base_gazebo/GazeboSystemInterface4WS4WD" />
+      </xacro:if>
+      <xacro:if value="${'4dv' in  mode or 'isaac' in mode}">
+        <xacro:property
+          name="simulation_hardware_plugin"
+          value="romea_mobile_base_simulation/GenericSimulationSystemInterface4WS4WD" />
+      </xacro:if>
+    </xacro:if>
+    <xacro:if value="${mode == 'live'}">
+      <xacro:property
+        name="live_hardware_plugin"
+        value="adap2e_hardware/Adap2eHardware" />
+    </xacro:if>
     <xacro:base_control mode="${mode}" base_name="${base_name}" />
   </xacro:macro>

File: adap2e_description/urdf/adap2e_fat.urdf.xacro (robot description, xacro)
@@ -8,13 +8,14 @@
   <xacro:arg name="ros_prefix" default="/adap2e/" />
   <xacro:include filename="$(find adap2e_description)/urdf/adap2e.xacro" />
-  <xacro:adap2e model="fat" mode="$(arg mode)" prefix="$(arg prefix)" />
-  <gazebo>
-    <plugin filename="libromea_gazebo_ros2_control.so" name="gazebo_ros2_control">
-      <ros2_control_config_file>$(arg ros2_control_config_urdf_file)</ros2_control_config_file>
-      <controller_manager_config_file>$(arg controller_manager_config_yaml_file)</controller_manager_config_file>
-      <ros>
-        <namespace>$(arg ros_prefix)$(arg base_name)</namespace>
-      </ros>
-    </plugin>
-  </gazebo>
+  <xacro:adap2e
+    model="fat"
+    mode="$(arg mode)"
+    prefix="$(arg prefix)" />
+  <xacro:include filename="$(find adap2e_description)/urdf/adap2e.simulation.xacro" />
+  <xacro:adap2e_simulation
+    mode="$(arg mode)"
+    base_name="$(arg base_name)"
+    ros_prefix="$(arg ros_prefix)"
+    ros2_control_config_urdf_file="$(arg ros2_control_config_urdf_file)"
+    controller_manager_config_yaml_file="$(arg controller_manager_config_yaml_file)" />
 </robot>

File: adap2e_description/urdf/adap2e_slim.urdf.xacro (robot description, xacro)
@@ -8,13 +8,14 @@
   <xacro:arg name="ros_prefix" default="/adap2e/" />
   <xacro:include filename="$(find adap2e_description)/urdf/adap2e.xacro" />
-  <xacro:adap2e model="slim" mode="$(arg mode)" prefix="$(arg prefix)" />
-  <gazebo>
-    <plugin filename="libromea_gazebo_ros2_control.so" name="gazebo_ros2_control">
-      <ros2_control_config_file>$(arg ros2_control_config_urdf_file)</ros2_control_config_file>
-      <controller_manager_config_file>$(arg controller_manager_config_yaml_file)</controller_manager_config_file>
-      <ros>
-        <namespace>$(arg ros_prefix)$(arg base_name)</namespace>
-      </ros>
-    </plugin>
-  </gazebo>
+  <xacro:adap2e
+    model="slim"
+    mode="$(arg mode)"
+    prefix="$(arg prefix)" />
+  <xacro:include filename="$(find adap2e_description)/urdf/adap2e.simulation.xacro" />
+  <xacro:adap2e_simulation
+    mode="$(arg mode)"
+    base_name="$(arg base_name)"
+    ros_prefix="$(arg ros_prefix)"
+    ros2_control_config_urdf_file="$(arg ros2_control_config_urdf_file)"
+    controller_manager_config_yaml_file="$(arg controller_manager_config_yaml_file)" />
 </robot>

Commit message: refactoring
Signed-off-by: Jean Laneurit <jean.laneurit@inrae.fr>

File: adap2e_description/ros2_control/adap2e.ros2_control.xacro (robot description, xacro)
@@ -5,5 +5,5 @@
       filename="$(find romea_mobile_base_description)/ros2_control/base4WS4WD.ros2_control.xacro" />
     <xacro:property name="conf" value="$(find adap2e_description)/config/adap2e_${model}.yaml" />
-    <xacro:property name="props" value="${load_yaml(conf)}" />
+    <xacro:property name="props" value="${xacro.load_yaml(conf)}" />
     <!-- Joint names -->
     <xacro:property name="front_left_wheel_steering_joint"

File: adap2e_description/urdf/adap2e.simulation.xacro (robot description, xacro)
@@ -4,5 +4,5 @@
     params="mode ros_prefix base_name controller_manager_config_yaml_file">
     <xacro:if value="${'simulation' in mode}">
-      <xacro:if value="${'gazebo' in  mode}">
+      <xacro:if value="${'gazebo_classic' in  mode}">
         <gazebo>
           <plugin filename="libgazebo_ros2_control.so" name="gazebo_ros2_control">
@@ -17,4 +17,18 @@
         </gazebo>
       </xacro:if>
+      <xacro:if value="${'gazebo_classic' not in  mode}">
+        <gazebo>
+          <plugin filename="gz_ros2_control-system"
+            name="gz_ros2_control::GazeboSimROS2ControlPlugin">
+            <robot_param>robot_description</robot_param>
+            <robot_param_node>ros2_control_description</robot_param_node>
+            <parameters>${controller_manager_config_yaml_file}</parameters>
+            <!-- <hold_joints>true</hold_joints> -->
+            <ros>
+              <namespace>${ros_prefix}${base_name}</namespace>
+            </ros>
+          </plugin>
+        </gazebo>
+      </xacro:if>
     </xacro:if>
   </xacro:macro>

File: adap2e_description/urdf/visual/chassis.xacro (robot description, xacro)
@@ -5,5 +5,6 @@
             <origin xyz="${-body_reference_x} 0 ${chassis_height}" rpy="0 0 ${M_PI/2.0}" />
             <geometry>
-                <mesh filename="package://adap2e_description/meshes/framev3_05.dae" />
+                <!-- <mesh filename="package://adap2e_description/meshes/framev3_05.dae" /> -->
+                <mesh filename="file://$(find adap2e_description)/meshes/framev3_05.dae" />
             </geometry>
             <material name="grey">

File: adap2e_description/urdf/visual/wheels.xacro (robot description, xacro)
@@ -5,5 +5,6 @@
             <origin xyz="0 0 0" rpy="0 ${orientation} 0" />
             <geometry>
-                <mesh filename="package://adap2e_description/meshes/wheel_02.dae" />
+                <!-- <mesh filename="package://adap2e_description/meshes/wheel_02.dae" /> -->
+                <mesh filename="file://$(find adap2e_description)/meshes/wheel_02.dae" />
             </geometry>
             <material name="black">

Commit message: add fake implement
Signed-off-by: Jean Laneurit <jean.laneurit@inrae.fr>

File: adap2e_description/ros2_control/adap2e.ros2_control.xacro (robot description, xacro)
@@ -44,4 +44,21 @@
           name="simulation_hardware_plugin"
           value="romea_mobile_base_gazebo/GazeboSystemInterface4WS4WD" />
+        <ros2_control name="${prefix}lift_arm" type="system">
+          <hardware>
+              <plugin>gz_ros2_control/GazeboSimSystem</plugin>
+          </hardware>
+          <joint name="${prefix}lift_arm_link_to_implement_link">
+              <param name="pos_kp">100000</param>
+              <param name="pos_ki">10.</param>
+              <param name="pos_kd">0</param>
+              <param name="pos_max_integral_error">10000</param>
+              <!-- <command_interface name="effort" /> -->
+              <command_interface name="position" />
+              <command_interface name="position_pid" />
+              <state_interface name="position" />
+              <state_interface name="velocity" />
+              <state_interface name="effort" />
+          </joint>
+        </ros2_control>
       </xacro:if>
       <xacro:if value="${'4dv' in  mode or 'isaac' in mode}">

File: adap2e_description/urdf/adap2e.xacro (robot description, xacro)
@@ -2,4 +2,5 @@
 <robot name="adap2e" xmlns:xacro="http://www.ros.org/wiki/xacro">
   <xacro:macro name="adap2e" params="model mode prefix">
+    <xacro:include filename="$(find romea_common_description)/urdf/inertia.xacro" />
     <xacro:include filename="$(find romea_mobile_base_description)/urdf/base4WS4WD.chassis.xacro" />
     <xacro:include filename="$(find adap2e_description)/urdf/visual/chassis.xacro" />
@@ -109,4 +110,22 @@
       <xacro:rear_right_wheel_visual />
     </xacro:chassis>
+    <link name="${prefix}lift_arm_link">
+      <xacro:box_inertia mass="0.1" lx="0.1" ly="0.1" lz="0.1"/>
+    </link>
+    <joint name="${prefix}base_footprint_to_lift_arm_link" type="fixed">
+        <origin xyz="-0.8 0.0 0.7" rpy="0.0 0.0 0.0" />
+        <parent link="${prefix}${base_footprint_link}" />
+        <child link="${prefix}lift_arm_link" />
+    </joint>
+    <link name="${prefix}implement_link">
+      <xacro:box_inertia mass="0.1" lx="0.1" ly="0.1" lz="0.1"/>
+    </link>
+    <joint name="${prefix}lift_arm_link_to_implement_link" type="prismatic">
+        <origin rpy="0 ${pi/2} 0" xyz="0 0 0" />
+        <parent link="${prefix}lift_arm_link" />
+        <child link="${prefix}implement_link" />
+        <dynamics damping="2000.0" friction="40." />
+        <limit effort="10000.0" lower="0" upper="1.0" velocity="0.1" />
+    </joint>
   </xacro:macro>
 </robot>
