Commit message: [description] update ros2 control xacro file
Signed-off-by: Jean Laneurit <jean.laneurit@inrae.fr>

File: adap2e_description/ros2_control/adap2e.ros2_control.xacro (robot description, xacro)
@@ -38,11 +38,9 @@
     <xacro:property name="maximal_wheel_speed"
       value="${props['wheels_speed_control']['command']['maximal_speed']}" />
-    <!-- simulation plugins -->
-    <xacro:if value="${'simulation' in mode}">
-      <xacro:if value="${'gazebo' in  mode}">
-        <xacro:property
-          name="simulation_hardware_plugin"
-          value="romea_mobile_base_gazebo/GazeboSystemInterface4WS4WD" />
-        <ros2_control name="${prefix}lift_arm" type="system">
+    <xacro:if value="${mode == 'simulation_gazebo'}">
+      <xacro:property
+        name="hardware_plugin"
+        value="romea_mobile_base_gazebo/GazeboSystemInterface" />
+      <ros2_control name="${prefix}lift_arm" type="system">
           <hardware>
               <plugin>gz_ros2_control/GazeboSimSystem</plugin>
@@ -53,5 +51,4 @@
               <param name="pos_kd">0</param>
               <param name="pos_max_integral_error">10000</param>
-              <!-- <command_interface name="effort" /> -->
               <command_interface name="position" />
               <command_interface name="position_pid" />
@@ -61,17 +58,24 @@
           </joint>
         </ros2_control>
-      </xacro:if>
-      <xacro:if value="${'4dv' in  mode or 'isaac' in mode}">
-        <xacro:property
-          name="simulation_hardware_plugin"
-          value="romea_mobile_base_simulation/GenericSimulationSystemInterface4WS4WD" />
-      </xacro:if>
+    </xacro:if>
+    <xacro:if value="${mode == 'simulation_gazebo_classic'}">
+      <xacro:property
+        name="hardware_plugin"
+        value="romea_mobile_base_gazebo/GazeboSystemInterface4WS4WD" />
+    </xacro:if>
+    <xacro:if value="${'4dv' in mode or 'isaac' in mode}">
+      <xacro:property
+        name="hardware_plugin"
+        value="romea_mobile_base_simulation/GenericSimulationSystemInterface" />
     </xacro:if>
     <xacro:if value="${mode ==  'live'}">
       <xacro:property
-        name="live_hardware_plugin"
+        name="hardware_plugin"
         value="adap2e_hardware/Adap2eHardware" />
     </xacro:if>
-    <xacro:base_control mode="${mode}" base_name="${base_name}" />
+    <xacro:base_control
+      mode="${mode}"
+      base_name="${base_name}"
+      hardware_plugin="${hardware_plugin}" />
   </xacro:macro>
 </robot>

Commit message: [description] Add properties.xacro to be included in adap2e.xacro and adap2e.ros2_control.xacro for better readability + remove three point hitch
Signed-off-by: Jean Laneurit <jean.laneurit@inrae.fr>

File: adap2e_description/ros2_control/adap2e.ros2_control.xacro (robot description, xacro)
@@ -2,60 +2,11 @@
 <robot name="adap2e" xmlns:xacro="http://www.ros.org/wiki/xacro">
   <xacro:macro name="adap2e_ros2_control" params="model mode prefix base_name">
-    <xacro:include
-      filename="$(find romea_mobile_base_description)/ros2_control/base4WS4WD.ros2_control.xacro" />
+    <xacro:include filename="$(find romea_mobile_base_description)/ros2_control/base4WS4WD.ros2_control.xacro" />
     <xacro:property name="conf" value="$(find adap2e_description)/config/adap2e_${model}.yaml" />
-    <xacro:property name="props" value="${xacro.load_yaml(conf)}" />
-    <!-- Joint names -->
-    <xacro:property name="front_left_wheel_steering_joint"
-      value="${props['joints']['front_left_wheel_steering_joint_name']}" />
-    <xacro:property name="front_right_wheel_steering_joint"
-      value="${props['joints']['front_right_wheel_steering_joint_name']}" />
-    <xacro:property name="rear_left_wheel_steering_joint"
-      value="${props['joints']['rear_left_wheel_steering_joint_name']}" />
-    <xacro:property name="rear_right_wheel_steering_joint"
-      value="${props['joints']['rear_right_wheel_steering_joint_name']}" />
-    <xacro:property name="front_left_wheel_spinning_joint"
-      value="${props['joints']['front_left_wheel_spinning_joint_name']}" />
-    <xacro:property name="front_right_wheel_spinning_joint"
-      value="${props['joints']['front_right_wheel_spinning_joint_name']}" />
-    <xacro:property name="rear_left_wheel_spinning_joint"
-      value="${props['joints']['rear_left_wheel_spinning_joint_name']}" />
-    <xacro:property name="rear_right_wheel_spinning_joint"
-      value="${props['joints']['rear_right_wheel_spinning_joint_name']}" />
-    <!-- Geometry -->
-    <xacro:property name="wheelbase"
-      value="${props['geometry']['axles_distance']}" />
-    <xacro:property name="front_track"
-      value="${props['geometry']['front_axle']['wheels_distance']}" />
-    <xacro:property name="rear_track"
-      value="${props['geometry']['rear_axle']['wheels_distance']}" />
-    <xacro:property name="front_wheel_radius"
-      value="${props['geometry']['front_axle']['wheels']['radius']}" />
-    <xacro:property name="rear_wheel_radius"
-      value="${props['geometry']['rear_axle']['wheels']['radius']}" />
-    <xacro:property name="maximal_wheel_steering_angle"
-      value="${props['wheels_steering_control']['command']['maximal_angle']}" />
-    <xacro:property name="maximal_wheel_speed"
-      value="${props['wheels_speed_control']['command']['maximal_speed']}" />
+    <xacro:include filename="$(find adap2e_description)/urdf/adap2e_properties.xacro" />
     <xacro:if value="${mode == 'simulation_gazebo'}">
       <xacro:property
         name="hardware_plugin"
         value="romea_mobile_base_gazebo/GazeboSystemInterface" />
-      <ros2_control name="${prefix}lift_arm" type="system">
-          <hardware>
-              <plugin>gz_ros2_control/GazeboSimSystem</plugin>
-          </hardware>
-          <joint name="${prefix}lift_arm_link_to_implement_link">
-              <param name="pos_kp">100000</param>
-              <param name="pos_ki">10.</param>
-              <param name="pos_kd">0</param>
-              <param name="pos_max_integral_error">10000</param>
-              <command_interface name="position" />
-              <command_interface name="position_pid" />
-              <state_interface name="position" />
-              <state_interface name="velocity" />
-              <state_interface name="effort" />
-          </joint>
-        </ros2_control>
     </xacro:if>
     <xacro:if value="${mode == 'simulation_gazebo_classic'}">
@@ -74,4 +25,5 @@
         value="adap2e_hardware/Adap2eHardware" />
     </xacro:if>
+    <xacro:base_control_model/>
     <xacro:base_control
       mode="${mode}"

File: adap2e_description/urdf/adap2e.xacro (robot description, xacro)
@@ -8,95 +8,5 @@
     <xacro:include filename="$(find adap2e_description)/urdf/visual/arms.xacro" />
     <xacro:property name="conf" value="$(find adap2e_description)/config/adap2e_${model}.yaml" />
-    <xacro:property name="props" value="${xacro.load_yaml(conf)}" />
-    <!-- Link names -->
-    <xacro:property name="base_link" value="${props['links']['base_link_name']}" />
-    <xacro:property name="base_footprint_link" value="${props['links']['base_footprint_link_name']}" />
-    <xacro:property name="inertial_link" value="${props['links']['inertial_link_name']}" />
-    <xacro:property name="front_left_wheel_steering_link"
-      value="${props['links']['front_left_wheel_steering_link_name']}" />
-    <xacro:property name="front_right_wheel_steering_link"
-      value="${props['links']['front_right_wheel_steering_link_name']}" />
-    <xacro:property name="rear_left_wheel_steering_link"
-      value="${props['links']['rear_left_wheel_steering_link_name']}" />
-    <xacro:property name="rear_right_wheel_steering_link"
-      value="${props['links']['rear_right_wheel_steering_link_name']}" />
-    <xacro:property name="front_left_wheel_spinning_link"
-      value="${props['links']['front_left_wheel_spinning_link_name']}" />
-    <xacro:property name="front_right_wheel_spinning_link"
-      value="${props['links']['front_right_wheel_spinning_link_name']}" />
-    <xacro:property name="rear_left_wheel_spinning_link"
-      value="${props['links']['rear_left_wheel_spinning_link_name']}" />
-    <xacro:property name="rear_right_wheel_spinning_link"
-      value="${props['links']['rear_right_wheel_spinning_link_name']}" />
-    <!-- Joint names -->
-    <xacro:property name="base_footprint_joint"
-      value="${props['joints']['base_footprint_joint_name']}" />
-    <xacro:property name="inertial_joint" value="${props['joints']['inertial_joint_name']}" />
-    <xacro:property name="front_left_wheel_steering_joint"
-      value="${props['joints']['front_left_wheel_steering_joint_name']}" />
-    <xacro:property name="front_right_wheel_steering_joint"
-      value="${props['joints']['front_right_wheel_steering_joint_name']}" />
-    <xacro:property name="rear_left_wheel_steering_joint"
-      value="${props['joints']['rear_left_wheel_steering_joint_name']}" />
-    <xacro:property name="rear_right_wheel_steering_joint"
-      value="${props['joints']['rear_right_wheel_steering_joint_name']}" />
-    <xacro:property name="front_left_wheel_spinning_joint"
-      value="${props['joints']['front_left_wheel_spinning_joint_name']}" />
-    <xacro:property name="front_right_wheel_spinning_joint"
-      value="${props['joints']['front_right_wheel_spinning_joint_name']}" />
-    <xacro:property name="rear_left_wheel_spinning_joint"
-      value="${props['joints']['rear_left_wheel_spinning_joint_name']}" />
-    <xacro:property name="rear_right_wheel_spinning_joint"
-      value="${props['joints']['rear_right_wheel_spinning_joint_name']}" />
-    <!-- Base Properties -->
-    <xacro:property name="aabb_length" value="${props['geometry']['aabb']['length']}" />
-    <xacro:property name="aabb_width" value="${props['geometry']['aabb']['width']}" />
-    <xacro:property name="aabb_height" value="${props['geometry']['aabb']['height']}" />
-    <xacro:property name="aabb_center_x" value="${props['geometry']['aabb']['center'][0]}" />
-    <xacro:property name="aabb_center_y" value="${props['geometry']['aabb']['center'][1]}" />
-    <xacro:property name="aabb_center_z" value="${props['geometry']['aabb']['center'][2]}" />
-    <xacro:property name="wheelbase" value="${props['geometry']['axles_distance']}" />
-    <xacro:property name="front_track" value="${props['geometry']['front_axle']['wheels_distance']}" />
-    <xacro:property name="rear_track" value="${props['geometry']['rear_axle']['wheels_distance']}" />
-    <xacro:property name="mass_base" value="${props['inertia']['mass']}" />
-    <xacro:property name="mass_center_x" value="${props['inertia']['center'][0]}" />
-    <xacro:property name="mass_center_y" value="${props['inertia']['center'][1]}" />
-    <xacro:property name="mass_center_z" value="${props['inertia']['center'][2]}" />
-    <xacro:property name="ground_clearance"
-      value="${props['geometry']['ground_clearance']}" />
-    <xacro:property name="body_reference_x"
-      value="${props['control_point'][0]}" />
-    <!-- Wheel Properties -->
-    <xacro:property name="front_wheel_x_offset" value="0.0" />
-    <xacro:property name="rear_wheel_x_offset" value="0.0" />
-    <xacro:property name="front_hub_carrier_offset"
-      value="${props['geometry']['front_axle']['wheels']['hub_carrier_offset']}" />
-    <xacro:property name="rear_hub_carrier_offset"
-      value="${props['geometry']['rear_axle']['wheels']['hub_carrier_offset']}" />
-    <xacro:property name="front_wheel_radius"
-      value="${props['geometry']['front_axle']['wheels']['radius']}" />
-    <xacro:property name="rear_wheel_radius"
-      value="${props['geometry']['rear_axle']['wheels']['radius']}" />
-    <xacro:property name="front_wheel_width"
-      value="${props['geometry']['front_axle']['wheels']['width']}" />
-    <xacro:property name="rear_wheel_width"
-      value="${props['geometry']['rear_axle']['wheels']['width']}" />
-    <xacro:property name="maximal_wheel_speed"
-      value="${props['wheels_speed_control']['command']['maximal_speed']}" />
-    <xacro:property name="chassis_height"
-      value="${min(front_wheel_radius,rear_wheel_radius)}" />
-    <xacro:property name="front_wheel_mass" value="10" />
-    <xacro:property name="rear_wheel_mass" value="10" />
-    <!-- Steering Properties -->
-    <xacro:property name="minimal_wheel_steering_angle"
-      value="-${props['wheels_steering_control']['command']['maximal_angle']}" />
-    <xacro:property name="maximal_wheel_steering_angle"
-      value="${props['wheels_steering_control']['command']['maximal_angle']}" />
-    <xacro:property name="front_wheel_steering_link_mass" value="20" />
-    <xacro:property name="front_wheel_steering_link_y" value="${front_hub_carrier_offset}" />
-    <xacro:property name="front_wheel_steering_link_xz" value="0.05" />
-    <xacro:property name="rear_wheel_steering_link_mass" value="20" />
-    <xacro:property name="rear_wheel_steering_link_y" value="${rear_hub_carrier_offset}" />
-    <xacro:property name="rear_wheel_steering_link_xz" value="0.05" />
+    <xacro:include filename="$(find adap2e_description)/urdf/adap2e_properties.xacro" />
     <xacro:chassis>
       <chassis_visuals>
@@ -112,22 +22,4 @@
       <xacro:rear_right_wheel_visual />
     </xacro:chassis>
-    <link name="${prefix}lift_arm_link">
-      <xacro:box_inertia mass="0.1" lx="0.1" ly="0.1" lz="0.1"/>
-    </link>
-    <joint name="${prefix}base_footprint_to_lift_arm_link" type="fixed">
-        <origin xyz="-0.8 0.0 0.7" rpy="0.0 0.0 0.0" />
-        <parent link="${prefix}${base_footprint_link}" />
-        <child link="${prefix}lift_arm_link" />
-    </joint>
-    <link name="${prefix}implement_link">
-      <xacro:box_inertia mass="0.1" lx="0.1" ly="0.1" lz="0.1"/>
-    </link>
-    <joint name="${prefix}lift_arm_link_to_implement_link" type="prismatic">
-        <origin rpy="0 ${pi/2} 0" xyz="0 0 0" />
-        <parent link="${prefix}lift_arm_link" />
-        <child link="${prefix}implement_link" />
-        <dynamics damping="2000.0" friction="40." />
-        <limit effort="10000.0" lower="0" upper="1.0" velocity="0.1" />
-    </joint>
   </xacro:macro>
 </robot>
